File: Shield Eagle Project/untitled.sch (EAGLE design)
At the start: 5 parts, among them IC1 MCP4922-E_P, J1 61PC6F, Q1 TLP222A-2_F_, U1 ARDUINOR3-BPLACE

Commit message: Add current limiting resistor for SSR to meet spec.
Parts:
- added R1: 130 ohm, adafruit:R-US_0207/7
Connections:
- new net N$3: Q1.CATHODE_1, Q1.CATHODE_2, R1.2
- net GND: now also R1.1; no longer Q1.CATHODE_1, Q1.CATHODE_2
Changed lines of the file:
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@@
 <?xml version="1.0" encoding="utf-8"?>
 <!DOCTYPE eagle SYSTEM "eagle.dtd">
-<eagle version="9.6.1">
+<eagle version="9.6.2">
 <drawing>
 <settings>
@@
 <part name="C1" library="rcl" library_urn="urn:adsk.eagle:library:334" deviceset="C-EU" device="050-024X044" package3d_urn="urn:adsk.eagle:package:23643/1" value="0.1uF"/>
 <part name="GND7" library="supply1" library_urn="urn:adsk.eagle:library:371" deviceset="GND" device=""/>
+<part name="R1" library="adafruit" deviceset="R-US_" device="0207/7" value="130 ohm"/>
 </parts>
 <sheets>
@@
 <attribute name="VALUE" x="-7.62" y="43.18" size="1.778" layer="96"/>
 </instance>
-<instance part="GND2" gate="1" x="76.2" y="27.94" smashed="yes">
-<attribute name="VALUE" x="73.66" y="25.4" size="1.778" layer="96"/>
+<instance part="GND2" gate="1" x="76.2" y="12.7" smashed="yes">
+<attribute name="VALUE" x="73.66" y="10.16" size="1.778" layer="96"/>
 </instance>
 <instance part="GND3" gate="1" x="114.3" y="58.42" smashed="yes">
@@
 <instance part="GND7" gate="1" x="170.18" y="91.44" smashed="yes">
 <attribute name="VALUE" x="167.64" y="88.9" size="1.778" layer="96"/>
+</instance>
+<instance part="R1" gate="G$1" x="76.2" y="22.86" smashed="yes" rot="R90">
+<attribute name="NAME" x="74.7014" y="19.05" size="1.778" layer="95" rot="R90"/>
+<attribute name="VALUE" x="79.502" y="19.05" size="1.778" layer="96" rot="R90"/>
 </instance>
 </instances>
@@
 </segment>
 <segment>
-<pinref part="Q1" gate="G$1" pin="CATHODE_2"/>
-<wire x1="76.2" y1="30.48" x2="76.2" y2="38.1" width="0.1524" layer="91"/>
-<wire x1="76.2" y1="38.1" x2="78.74" y2="38.1" width="0.1524" layer="91"/>
-<pinref part="Q1" gate="G$1" pin="CATHODE_1"/>
-<wire x1="78.74" y1="43.18" x2="76.2" y2="43.18" width="0.1524" layer="91"/>
-<wire x1="76.2" y1="43.18" x2="76.2" y2="38.1" width="0.1524" layer="91"/>
-<junction x="76.2" y="38.1"/>
-<pinref part="GND2" gate="1" pin="GND"/>
-</segment>
-<segment>
 <wire x1="114.3" y1="60.96" x2="114.3" y2="76.2" width="0.1524" layer="91"/>
 <pinref part="IC1" gate="G$1" pin="AVSS"/>
@@
 <pinref part="C1" gate="G$1" pin="2"/>
 <pinref part="GND7" gate="1" pin="GND"/>
+</segment>
+<segment>
+<pinref part="GND2" gate="1" pin="GND"/>
+<pinref part="R1" gate="G$1" pin="1"/>
+<wire x1="76.2" y1="15.24" x2="76.2" y2="17.78" width="0.1524" layer="91"/>
 </segment>
 </net>
@@
 </segment>
 </net>
+<net name="N$3" class="0">
+<segment>
+<pinref part="Q1" gate="G$1" pin="CATHODE_2"/>
+<wire x1="76.2" y1="38.1" x2="78.74" y2="38.1" width="0.1524" layer="91"/>
+<pinref part="Q1" gate="G$1" pin="CATHODE_1"/>
+<wire x1="78.74" y1="43.18" x2="76.2" y2="43.18" width="0.1524" layer="91"/>
+<wire x1="76.2" y1="43.18" x2="76.2" y2="38.1" width="0.1524" layer="91"/>
+<pinref part="R1" gate="G$1" pin="2"/>
+<wire x1="76.2" y1="27.94" x2="76.2" y2="38.1" width="0.1524" layer="91"/>
+<junction x="76.2" y="38.1"/>
+</segment>
+</net>

Commit message: Using individual resistors between opto isolator and ground to avoid under current conditions that might have happened otherwise.
Parts:
- added R2: 130 ohm, adafruit:R-US_0207/7
Connections:
- new net N$6: Q1.CATHODE_1, R2.2
- net GND: now also R2.1
- net N$3: no longer Q1.CATHODE_1
Changed lines of the file:
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@@
 <part name="GND7" library="supply1" library_urn="urn:adsk.eagle:library:371" deviceset="GND" device=""/>
 <part name="R1" library="adafruit" deviceset="R-US_" device="0207/7" value="130 ohm"/>
+<part name="R2" library="adafruit" deviceset="R-US_" device="0207/7" value="130 ohm"/>
+<part name="GND8" library="supply1" library_urn="urn:adsk.eagle:library:371" deviceset="GND" device=""/>
 </parts>
 <sheets>
@@
 <attribute name="VALUE" x="79.502" y="19.05" size="1.778" layer="96" rot="R90"/>
 </instance>
+<instance part="R2" gate="G$1" x="68.58" y="22.86" smashed="yes" rot="R90">
+<attribute name="NAME" x="67.0814" y="19.05" size="1.778" layer="95" rot="R90"/>
+<attribute name="VALUE" x="71.882" y="19.05" size="1.778" layer="96" rot="R90"/>
+</instance>
+<instance part="GND8" gate="1" x="68.58" y="12.7" smashed="yes">
+<attribute name="VALUE" x="66.04" y="10.16" size="1.778" layer="96"/>
+</instance>
 </instances>
 <busses>
@@
 <pinref part="R1" gate="G$1" pin="1"/>
 <wire x1="76.2" y1="15.24" x2="76.2" y2="17.78" width="0.1524" layer="91"/>
+</segment>
+<segment>
+<pinref part="GND8" gate="1" pin="GND"/>
+<pinref part="R2" gate="G$1" pin="1"/>
+<wire x1="68.58" y1="15.24" x2="68.58" y2="17.78" width="0.1524" layer="91"/>
 </segment>
 </net>
@@
 <pinref part="Q1" gate="G$1" pin="CATHODE_2"/>
 <wire x1="76.2" y1="38.1" x2="78.74" y2="38.1" width="0.1524" layer="91"/>
-<pinref part="Q1" gate="G$1" pin="CATHODE_1"/>
-<wire x1="78.74" y1="43.18" x2="76.2" y2="43.18" width="0.1524" layer="91"/>
-<wire x1="76.2" y1="43.18" x2="76.2" y2="38.1" width="0.1524" layer="91"/>
 <pinref part="R1" gate="G$1" pin="2"/>
 <wire x1="76.2" y1="27.94" x2="76.2" y2="38.1" width="0.1524" layer="91"/>
-<junction x="76.2" y="38.1"/>
-</segment>
-</net>
+</segment>
+</net>
+<net name="N$6" class="0">
+<segment>
+<pinref part="R2" gate="G$1" pin="2"/>
+<wire x1="68.58" y1="27.94" x2="68.58" y2="33.02" width="0.1524" layer="91"/>
+<wire x1="68.58" y1="33.02" x2="73.66" y2="33.02" width="0.1524" layer="91"/>
+<wire x1="73.66" y1="33.02" x2="73.66" y2="43.18" width="0.1524" layer="91"/>
+<pinref part="Q1" gate="G$1" pin="CATHODE_1"/>
+<wire x1="73.66" y1="43.18" x2="78.74" y2="43.18" width="0.1524" layer="91"/>
+</segment>
+</net>
